File: sockets-split.sch (KiCad schematic (older format))
At the start: 57 parts, among them J1 LED, J2 Conn_01x01, J3 MJ-4PP-9, J4 Conn_01x01, SW1 RESET_SW, SW10 SW_PUSH, SW11 SW_PUSH, SW12 SW_PUSH, SW13 SW_PUSH, SW14 SW_PUSH, SW15 SW_PUSH, SW16 SW_PUSH, SW17 SW_PUSH, SW18 SW_PUSH, SW19 SW_PUSH, SW2 SW_PUSH, SW20 SW_PUSH, SW21 SW_PUSH, SW22 SW_PUSH, SW23 SW_PUSH, SW24 SW_PUSH, SW25 SW_PUSH, SW3 SW_PUSH, SW4 SW_PUSH, SW5 SW_PUSH, SW6 SW_PUSH, SW7 SW_PUSH, SW8 SW_PUSH, SW9 SW_PUSH, U1 ProMicro

Commit message: Add LEDをTHTのフットプリントにした
Parts:
- J1: footprint kbd:StripLED_rev -> kbd:StripLED_THT
- JP1: footprint kbd:Jumper -> kbd:JPC2
Changed lines of the file:
@@
 F 0 "J1" H 3470 1575 50  0000 C CNN
 F 1 "LED" H 3470 1666 50  0000 C CNN
-F 2 "kbd:StripLED_rev" H 3550 1900 50  0001 C CNN
+F 2 "kbd:StripLED_THT" H 3550 1900 50  0001 C CNN
 F 3 "~" H 3550 1900 50  0001 C CNN
 	1    3550 1900
@@
 F 0 "JP1" H 4450 2640 50  0000 C CNN
 F 1 "Jumper_NC_Small" H 4450 2731 50  0000 C CNN
-F 2 "kbd:Jumper" H 4450 2825 50  0001 C CNN
+F 2 "kbd:JPC2" H 4450 2825 50  0001 C CNN
 F 3 "~" H 4450 2825 50  0001 C CNN
 	1    4450 2825

Commit message: Fix ネットリスト修正
Parts:
- P1: renamed from J2; value Conn_01x01 -> i2c-pin
- P2: renamed from J4; value Conn_01x01 -> i2c-pin
- renumbered J3 to J2
Changed lines of the file:
@@
 	3800 2000 3800 2050
 $Comp
-L kbd:MJ-4PP-9 J3
+L kbd:MJ-4PP-9 J2
 U 1 1 5C2E0F41
 P 3450 2750
-F 0 "J3" H 3480 3026 50  0000 C CNN
+F 0 "J2" H 3480 3026 50  0000 C CNN
 F 1 "MJ-4PP-9" H 3480 2935 50  0000 C CNN
 F 2 "kbd:MJ-4PP-9" H 3725 2925 50  0001 C CNN
@@
 $EndComp
 $Comp
-L Connector_Generic:Conn_01x01 J4
+L Connector_Generic:Conn_01x01 P2
 U 1 1 5C32CF8C
 P 4050 3025
-F 0 "J4" V 3923 3105 50  0000 L CNN
-F 1 "Conn_01x01" V 4014 3105 50  0000 L CNN
+F 0 "P2" V 3923 3105 50  0000 L CNN
+F 1 "i2c-pin" V 4014 3105 50  0000 L CNN
 F 2 "kbd:1pin_conn" H 4050 3025 50  0001 C CNN
 F 3 "~" H 4050 3025 50  0001 C CNN
@@
 $EndComp
 $Comp
-L Connector_Generic:Conn_01x01 J2
+L Connector_Generic:Conn_01x01 P1
 U 1 1 5C32F9D9
 P 4050 2400
-F 0 "J2" V 4016 2312 50  0000 R CNN
-F 1 "Conn_01x01" V 3925 2312 50  0000 R CNN
+F 0 "P1" V 4016 2312 50  0000 R CNN
+F 1 "i2c-pin" V 3925 2312 50  0000 R CNN
 F 2 "kbd:1pin_conn" H 4050 2400 50  0001 C CNN
 F 3 "~" H 4050 2400 50  0001 C CNN

Commit message: 再配線開始
Parts:
- U1: footprint kbd:ProMicro_v2_one -> kbd:ProMicro_v2
Changed lines of the file:
@@
 F 0 "U1" H 2000 3087 60  0000 C CNN
 F 1 "ProMicro" H 2000 2981 60  0000 C CNN
-F 2 "kbd:ProMicro_v2_one" H 2100 1000 60  0001 C CNN
+F 2 "kbd:ProMicro_v2" H 2100 1000 60  0001 C CNN
 F 3 "" H 2100 1000 60  0000 C CNN
 	1    2000 2050

Commit message: Fix module & draw case line
Parts:
- U1: footprint kbd:ProMicro_v2 -> kbd:ProMicro_v2_ura_pcb_for_sockets_split
Changed lines of the file:
@@
 F 0 "U1" H 2000 3087 60  0000 C CNN
 F 1 "ProMicro" H 2000 2981 60  0000 C CNN
-F 2 "kbd:ProMicro_v2" H 2100 1000 60  0001 C CNN
+F 2 "kbd:ProMicro_v2_ura_pcb_for_sockets_split" H 2100 1000 60  0001 C CNN
 F 3 "" H 2100 1000 60  0000 C CNN
 	1    2000 2050
