File: sockets-split-top-plate/sockets-split-top-plate.kicad_pcb (KiCad board)
At the start: 2 copper layers, 137.9 x 84.6 mm, 0 parts

Commit message: 穴を修正してみた
Parts:
- added Ref**: Val**, kbd:HOLE, F.Cu at (93.4, 57.5)
- added Ref**: Val**, kbd:HOLE, F.Cu at (209.6, 58.2)
- added Ref**: Val**, kbd:HOLE, F.Cu at (195.9, 135.8)
- added Ref**: Val**, kbd:HOLE, F.Cu at (79.6, 136.6)
Routing:
- net (no net): vias 4 -> 0
Changed lines of the file:
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@@
-(kicad_pcb (version 20171130) (host pcbnew "(5.0.2)-1")
+(kicad_pcb (version 20171130) (host pcbnew "(5.0.0-3-g5ebb6b6)")
   (general
     (thickness 1.6)
-    (drawings 140)
-    (tracks 4)
+    (drawings 131)
+    (tracks 0)
     (zones 0)
-    (modules 0)
+    (modules 4)
     (nets 1)
   )
@@
     (mod_text_size 1 1)
     (mod_text_width 0.15)
-    (pad_size 1.524 1.524)
-    (pad_drill 0.762)
+    (pad_size 2.2 2.2)
+    (pad_drill 2)
     (pad_to_mask_clearance 0.051)
     (solder_mask_min_width 0.25)
@@
       (drillshape 0)
       (scaleselection 1)
-      (outputdirectory "../../../../Desktop/sockets-split-1.2/sockets-split-top/"))
+      (outputdirectory "../../../../Desktop/sockets-split/sockets-split-top/"))
   )
   (net 0 "")
@@
     (uvia_drill 0.1)
   )
-  (gr_circle (center 211.07925 56.81) (end 212.28 56.81) (layer F.Mask) (width 0.2))
-  (gr_circle (center 211.07925 56.81) (end 212.28 56.81) (layer B.Mask) (width 0.2))
-  (gr_circle (center 197.19925 137.17) (end 198.4 137.17) (layer B.Mask) (width 0.2))
-  (gr_circle (center 197.19925 137.17) (end 198.4 137.17) (layer F.Mask) (width 0.2))
-  (gr_circle (center 77.42 137.17) (end 78.62075 137.17) (layer B.Mask) (width 0.2))
-  (gr_circle (center 77.42 137.17) (end 78.62075 137.17) (layer F.Mask) (width 0.2))
-  (gr_circle (center 92.27925 56.8) (end 93.48 56.8) (layer B.Mask) (width 0.2))
-  (gr_circle (center 92.289251 56.81) (end 93.490001 56.81) (layer F.Mask) (width 0.2))
-  (dimension 84.605111 (width 0.3) (layer F.SilkS)
-    (gr_text "84.605 mm" (at 51.74 97.072555 270) (layer F.SilkS)
-      (effects (font (size 1.5 1.5) (thickness 0.3)))
-    )
-    (feature1 (pts (xy 97.55 139.375111) (xy 53.253579 139.375111)))
-    (feature2 (pts (xy 97.55 54.77) (xy 53.253579 54.77)))
-    (crossbar (pts (xy 53.84 54.77) (xy 53.84 139.375111)))
-    (arrow1a (pts (xy 53.84 139.375111) (xy 53.253579 138.248607)))
-    (arrow1b (pts (xy 53.84 139.375111) (xy 54.426421 138.248607)))
-    (arrow2a (pts (xy 53.84 54.77) (xy 53.253579 55.896504)))
-    (arrow2b (pts (xy 53.84 54.77) (xy 54.426421 55.896504)))
-  )
-  (dimension 137.77144 (width 0.3) (layer F.SilkS)
-    (gr_text "137.771 mm" (at 144.37572 165.15) (layer F.SilkS)
+  (module kbd:HOLE (layer F.Cu)
+    (at 93.39 57.54)
+    (descr "Mounting Hole 2.2mm, no annular, M2")
+    (tags "mounting hole 2.2mm no annular m2")
+    (attr virtual)
+    (fp_text reference Ref** (at 0 -3.2) (layer F.Fab)
+      (effects (font (size 1 1) (thickness 0.15)))
+    )
+    (fp_text value Val** (at 0 3.2) (layer F.Fab)
+      (effects (font (size 1 1) (thickness 0.15)))
+    )
+    (fp_circle (center 0 0) (end 2.45 0) (layer F.CrtYd) (width 0.05))
+    (fp_circle (center 0 0) (end 2.2 0) (layer Cmts.User) (width 0.15))
+    (fp_text user %R (at 0.3 0) (layer F.Fab)
+      (effects (font (size 1 1) (thickness 0.15)))
+    )
+    (pad "" np_thru_hole circle (at -1.1 -0.73) (size 2.2 2.2) (drill 2) (layers *.Cu *.Mask))
+  )
+  (module kbd:HOLE (layer F.Cu)
+    (at 209.62 58.24)
+    (descr "Mounting Hole 2.2mm, no annular, M2")
+    (tags "mounting hole 2.2mm no annular m2")
+    (attr virtual)
+    (fp_text reference Ref** (at 0 -3.2) (layer F.Fab)
+      (effects (font (size 1 1) (thickness 0.15)))
+    )
+    (fp_text value Val** (at 0 3.2) (layer F.Fab)
+      (effects (font (size 1 1) (thickness 0.15)))
+    )
+    (fp_circle (center 0 0) (end 2.45 0) (layer F.CrtYd) (width 0.05))
+    (fp_circle (center 0 0) (end 2.2 0) (layer Cmts.User) (width 0.15))
+    (fp_text user %R (at 0.3 0) (layer F.Fab)
+      (effects (font (size 1 1) (thickness 0.15)))
+    )
+    (pad "" np_thru_hole circle (at 1.46 -1.43) (size 2.2 2.2) (drill 2) (layers *.Cu *.Mask))
+  )
+  (module kbd:HOLE (layer F.Cu)
+    (at 195.93 135.8)
+    (descr "Mounting Hole 2.2mm, no annular, M2")
+    (tags "mounting hole 2.2mm no annular m2")
+    (attr virtual)
+    (fp_text reference Ref** (at 0 -3.2) (layer F.Fab)
+      (effects (font (size 1 1) (thickness 0.15)))
+    )
+    (fp_text value Val** (at 0 3.2) (layer F.Fab)
+      (effects (font (size 1 1) (thickness 0.15)))
+    )
+    (fp_circle (center 0 0) (end 2.45 0) (layer F.CrtYd) (width 0.05))
+    (fp_circle (center 0 0) (end 2.2 0) (layer Cmts.User) (width 0.15))
+    (fp_text user %R (at 0.3 0) (layer F.Fab)
+      (effects (font (size 1 1) (thickness 0.15)))
+    )
+    (pad "" np_thru_hole circle (at 1.27 1.367) (size 2.2 2.2) (drill 2) (layers *.Cu *.Mask))
+  )
+  (module kbd:HOLE (layer F.Cu)
+    (at 79.62 136.63)
+    (descr "Mounting Hole 2.2mm, no annular, M2")
+    (tags "mounting hole 2.2mm no annular m2")
+    (attr virtual)
+    (fp_text reference Ref** (at 0 -3.2) (layer F.Fab)
+      (effects (font (size 1 1) (thickness 0.15)))
+    )
+    (fp_text value Val** (at 0 3.2) (layer F.Fab)
+      (effects (font (size 1 1) (thickness 0.15)))
+    )
+    (fp_circle (center 0 0) (end 2.45 0) (layer F.CrtYd) (width 0.05))
+    (fp_circle (center 0 0) (end 2.2 0) (layer Cmts.User) (width 0.15))
+    (fp_text user %R (at 0.3 0) (layer F.Fab)
+      (effects (font (size 1 1) (thickness 0.15)))
+    )
+    (pad "" np_thru_hole circle (at -2.2 0.537) (size 2.2 2.2) (drill 2) (layers *.Cu *.Mask))
+  )
+  (dimension 137.77144 (width 0.3) (layer Dwgs.User)
+    (gr_text "137.771 mm" (at 144.37572 165.15) (layer Dwgs.User)
       (effects (font (size 1.5 1.5) (thickness 0.3)))
     )
@@
   (gr_line (start 76.607796 139.377551) (end 198.066532 139.377551) (layer Edge.Cuts) (width 0.2))
   (gr_line (start 213.36 55.88) (end 213.357244 80.89) (layer Edge.Cuts) (width 0.2))
-  (via (at 211.08 56.81) (size 2.2) (drill 2) (layers F.Cu B.Cu) (net 0))
-  (via (at 197.2 137.167) (size 2.2) (drill 2) (layers F.Cu B.Cu) (net 0))
-  (via (at 77.42 137.167) (size 2.2) (drill 2) (layers F.Cu B.Cu) (net 0))
-  (via (at 92.29 56.81) (size 2.2) (drill 2) (layers F.Cu B.Cu) (net 0))
 )
