File: sockets-split-top-plate/sockets-split-top-plate.kicad_pcb (KiCad board)
At the start: 2 copper layers, 137.9 x 85.2 mm, 0 parts

Commit message: Update docs
Parts:
- added Ref**: Val**, kbd:HOLE, F.Cu at (93.4, 57.5)
- added Ref**: Val**, kbd:HOLE, F.Cu at (209.6, 58.2)
- added Ref**: Val**, kbd:HOLE, F.Cu at (195.9, 135.8)
- added Ref**: Val**, kbd:HOLE, F.Cu at (79.6, 136.6)
Routing:
- net (no net): vias 4 -> 0
Other:
- board size 137.9 x 85.2 mm -> 137.9 x 84.6 mm
Changed lines of the file:
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@@
-(kicad_pcb (version 20171130) (host pcbnew "(5.0.2)-1")
+(kicad_pcb (version 20171130) (host pcbnew "(5.0.0-3-g5ebb6b6)")
   (general
     (thickness 1.6)
-    (drawings 132)
-    (tracks 4)
+    (drawings 131)
+    (tracks 0)
     (zones 0)
-    (modules 0)
+    (modules 4)
     (nets 1)
   )
@@
     (mod_text_size 1 1)
     (mod_text_width 0.15)
-    (pad_size 1.524 1.524)
-    (pad_drill 0.762)
+    (pad_size 2.2 2.2)
+    (pad_drill 2)
     (pad_to_mask_clearance 0.051)
     (solder_mask_min_width 0.25)
@@
       (drillshape 0)
       (scaleselection 1)
-      (outputdirectory "../../../../Desktop/sockets-split-1.1/sockets-split-top/"))
+      (outputdirectory "../../../../Desktop/sockets-split/sockets-split-top/"))
   )
   (net 0 "")
@@
     (uvia_drill 0.1)
   )
-  (dimension 85.160366 (width 0.3) (layer F.SilkS)
-    (gr_text "85.160 mm" (at 63.87 97.390183 270) (layer F.SilkS)
-      (effects (font (size 1.5 1.5) (thickness 0.3)))
-    )
-    (feature1 (pts (xy 85.45 139.970366) (xy 65.383579 139.970366)))
-    (feature2 (pts (xy 85.45 54.81) (xy 65.383579 54.81)))
-    (crossbar (pts (xy 65.97 54.81) (xy 65.97 139.970366)))
-    (arrow1a (pts (xy 65.97 139.970366) (xy 65.383579 138.843862)))
-    (arrow1b (pts (xy 65.97 139.970366) (xy 66.556421 138.843862)))
-    (arrow2a (pts (xy 65.97 54.81) (xy 65.383579 55.936504)))
-    (arrow2b (pts (xy 65.97 54.81) (xy 66.556421 55.936504)))
-  )
-  (dimension 137.77144 (width 0.3) (layer F.SilkS)
-    (gr_text "137.771 mm" (at 144.37572 165.15) (layer F.SilkS)
+  (module kbd:HOLE (layer F.Cu)
+    (at 93.39 57.54)
+    (descr "Mounting Hole 2.2mm, no annular, M2")
+    (tags "mounting hole 2.2mm no annular m2")
+    (attr virtual)
+    (fp_text reference Ref** (at 0 -3.2) (layer F.Fab)
+      (effects (font (size 1 1) (thickness 0.15)))
+    )
+    (fp_text value Val** (at 0 3.2) (layer F.Fab)
+      (effects (font (size 1 1) (thickness 0.15)))
+    )
+    (fp_circle (center 0 0) (end 2.45 0) (layer F.CrtYd) (width 0.05))
+    (fp_circle (center 0 0) (end 2.2 0) (layer Cmts.User) (width 0.15))
+    (fp_text user %R (at 0.3 0) (layer F.Fab)
+      (effects (font (size 1 1) (thickness 0.15)))
+    )
+    (pad "" np_thru_hole circle (at -1.1 -0.73) (size 2.2 2.2) (drill 2) (layers *.Cu *.Mask))
+  )
+  (module kbd:HOLE (layer F.Cu)
+    (at 209.62 58.24)
+    (descr "Mounting Hole 2.2mm, no annular, M2")
+    (tags "mounting hole 2.2mm no annular m2")
+    (attr virtual)
+    (fp_text reference Ref** (at 0 -3.2) (layer F.Fab)
+      (effects (font (size 1 1) (thickness 0.15)))
+    )
+    (fp_text value Val** (at 0 3.2) (layer F.Fab)
+      (effects (font (size 1 1) (thickness 0.15)))
+    )
+    (fp_circle (center 0 0) (end 2.45 0) (layer F.CrtYd) (width 0.05))
+    (fp_circle (center 0 0) (end 2.2 0) (layer Cmts.User) (width 0.15))
+    (fp_text user %R (at 0.3 0) (layer F.Fab)
+      (effects (font (size 1 1) (thickness 0.15)))
+    )
+    (pad "" np_thru_hole circle (at 1.46 -1.43) (size 2.2 2.2) (drill 2) (layers *.Cu *.Mask))
+  )
+  (module kbd:HOLE (layer F.Cu)
+    (at 195.93 135.8)
+    (descr "Mounting Hole 2.2mm, no annular, M2")
+    (tags "mounting hole 2.2mm no annular m2")
+    (attr virtual)
+    (fp_text reference Ref** (at 0 -3.2) (layer F.Fab)
+      (effects (font (size 1 1) (thickness 0.15)))
+    )
+    (fp_text value Val** (at 0 3.2) (layer F.Fab)
+      (effects (font (size 1 1) (thickness 0.15)))
+    )
+    (fp_circle (center 0 0) (end 2.45 0) (layer F.CrtYd) (width 0.05))
+    (fp_circle (center 0 0) (end 2.2 0) (layer Cmts.User) (width 0.15))
+    (fp_text user %R (at 0.3 0) (layer F.Fab)
+      (effects (font (size 1 1) (thickness 0.15)))
+    )
+    (pad "" np_thru_hole circle (at 1.27 1.367) (size 2.2 2.2) (drill 2) (layers *.Cu *.Mask))
+  )
+  (module kbd:HOLE (layer F.Cu)
+    (at 79.62 136.63)
+    (descr "Mounting Hole 2.2mm, no annular, M2")
+    (tags "mounting hole 2.2mm no annular m2")
+    (attr virtual)
+    (fp_text reference Ref** (at 0 -3.2) (layer F.Fab)
+      (effects (font (size 1 1) (thickness 0.15)))
+    )
+    (fp_text value Val** (at 0 3.2) (layer F.Fab)
+      (effects (font (size 1 1) (thickness 0.15)))
+    )
+    (fp_circle (center 0 0) (end 2.45 0) (layer F.CrtYd) (width 0.05))
+    (fp_circle (center 0 0) (end 2.2 0) (layer Cmts.User) (width 0.15))
+    (fp_text user %R (at 0.3 0) (layer F.Fab)
+      (effects (font (size 1 1) (thickness 0.15)))
+    )
+    (pad "" np_thru_hole circle (at -2.2 0.537) (size 2.2 2.2) (drill 2) (layers *.Cu *.Mask))
+  )
+  (dimension 137.77144 (width 0.3) (layer Dwgs.User)
+    (gr_text "137.771 mm" (at 144.37572 165.15) (layer Dwgs.User)
       (effects (font (size 1.5 1.5) (thickness 0.3)))
     )
@@
   (gr_arc (start 202.72 119.04) (end 202.72 120.13) (angle -93.34194386) (layer Edge.Cuts) (width 0.2))
   (gr_arc (start 200.27 121.23) (end 200.27 120.14) (angle -93.34194386) (layer Edge.Cuts) (width 0.2))
-  (gr_arc (start 198.08 138.91) (end 198.08 140) (angle -90) (layer Edge.Cuts) (width 0.2))
-  (gr_arc (start 76.57 138.91) (end 75.48 138.91) (angle -90) (layer Edge.Cuts) (width 0.2))
+  (gr_arc (start 198.07 138.3) (end 198.07 139.39) (angle -90) (layer Edge.Cuts) (width 0.2))
+  (gr_arc (start 76.57 138.29) (end 75.48 138.29) (angle -90) (layer Edge.Cuts) (width 0.2))
   (gr_arc (start 79.33 111.33) (end 79.33 112.42) (angle -93.3) (layer Edge.Cuts) (width 0.2))
   (gr_arc (start 76.58 113.51) (end 76.58 112.42) (angle -93.3) (layer Edge.Cuts) (width 0.2))
@@
   (gr_line (start 196.815274 99.108886) (end 196.815274 113.10717) (layer Edge.Cuts) (width 0.2))
   (gr_line (start 130.428628 80.058886) (end 144.427774 80.058886) (layer Edge.Cuts) (width 0.2))
-  (gr_line (start 199.184121 121.258266) (end 199.17 138.94) (layer Edge.Cuts) (width 0.2))
-  (gr_line (start 75.490207 113.531606) (end 75.48 138.92) (layer Edge.Cuts) (width 0.2))
+  (gr_line (start 199.184121 121.258266) (end 199.17 138.317) (layer Edge.Cuts) (width 0.2))
+  (gr_line (start 75.490207 113.531606) (end 75.48 138.297) (layer Edge.Cuts) (width 0.2))
   (gr_line (start 86.473172 74.320735) (end 89.16448 74.320735) (layer Edge.Cuts) (width 0.2))
   (gr_line (start 163.477774 80.058886) (end 163.477774 94.056998) (layer Edge.Cuts) (width 0.2))
@@
   (gr_line (start 208.42938 83.156716) (end 208.430758 99.978428) (layer Edge.Cuts) (width 0.2))
   (gr_line (start 212.244478 54.763445) (end 91.366413 54.774813) (layer Edge.Cuts) (width 0.2))
-  (gr_line (start 76.607796 140.000551) (end 198.066532 140.000551) (layer Edge.Cuts) (width 0.2))
+  (gr_line (start 76.607796 139.377551) (end 198.066532 139.377551) (layer Edge.Cuts) (width 0.2))
   (gr_line (start 213.36 55.88) (end 213.357244 80.89) (layer Edge.Cuts) (width 0.2))
-  (via (at 211.08 56.81) (size 2.2) (drill 2) (layers F.Cu B.Cu) (net 0))
-  (via (at 197.2 137.79) (size 2.2) (drill 2) (layers F.Cu B.Cu) (net 0))
-  (via (at 77.42 137.79) (size 2.2) (drill 2) (layers F.Cu B.Cu) (net 0))
-  (via (at 92.29 56.81) (size 2.2) (drill 2) (layers F.Cu B.Cu) (net 0))
 )
